Commit message: remove jitter

File: simultation_ws/src/arm_descrption/urdf/arm.xacro (robot description, xacro)
@@ -3,7 +3,7 @@
     <link name="base_link">
         <inertial>
-        <mass value="6"/>
+        <mass value="10000"/>
         <origin rpy="0 0 0" xyz="0 0 0"/>
-        <inertia ixx="0.0395416666667" ixy="0" ixz="0" iyy="0.106208333333" iyz="0" izz="0.106208333333"/>
+        <inertia ixx="7708" ixy="0" ixz="0" iyy="7708" iyz="0" izz="15000"/>
         </inertial>
         <!-- body -->

Commit message: end-effector

File: simultation_ws/src/arm_descrption/urdf/arm.xacro (robot description, xacro)
@@ -122,4 +122,28 @@
         </visual>
     </link>
+    <link name="third_link">
+    <inertial>
+        <mass value="1"/>
+        <origin rpy="0 0 0" xyz="-0.53 0 1"/>
+        <inertia ixx="0.0395416666667" ixy="0" ixz="0" iyy="0.106208333333" iyz="0" izz="0.106208333333"/>
+        </inertial>
+        <!-- body -->
+        <collision name="collision_chassis">
+        <geometry>
+            <box size="0.25 0.25 0.25"/>
+        </geometry>
+        </collision>
+        <visual>
+        <origin rpy="0 0 0" xyz="0 0 0"/>
+        <geometry>
+            <box size="0.25 0.25 0.25"/>
+        </geometry>
+        </visual>
+    </link>
+    <joint name="end" type="fixed">
+        <origin rpy="0 0 0" xyz="0 0 2.5"/>
+        <parent link="second_link"/>
+        <child link="third_link"/>
+    </joint>
      <gazebo>
     <plugin name="gazebo_ros_control" filename="libgazebo_ros_control.so">

Commit message: done

File: simultation_ws/src/arm_descrption/urdf/arm.xacro (robot description, xacro)
@@ -23,5 +23,5 @@
         <axis xyz="0 0 1" />
         <limit effort="1000.0" lower="-3.14" upper="3.14" velocity="0.5" />
-        <origin rpy="0 0 0" xyz="0 0 0.5"/>
+        <origin rpy="0 0 0" xyz="0 0 0.45"/>
         <parent link="base_link"/>
         <child link="base_rotation"/>
@@ -39,18 +39,18 @@
     <link name="base_rotation">
          <inertial>
-            <origin xyz="0 0 0.2" rpy="0 0 0" />
+            <origin xyz="0 0 0" rpy="0 0 0" />
             <mass value="1" />
-            <xacro:cylinder_inertia mass="1" r="0.5" l="0.4" />
+            <xacro:cylinder_inertia mass="1" r="0.5" l="0.5" />
         </inertial>
          <collision>
-            <origin xyz="0 0 0.2" rpy="0 0 0"/>
+            <origin xyz="0 0 0" rpy="0 0 0"/>
             <geometry>
-                <cylinder radius="0.5" length="0.4"/>
+                <cylinder radius="0.5" length="0.5"/>
             </geometry>
         </collision>
         <visual>
-            <origin rpy="0 0 0" xyz="0 0 0.2"/>
+            <origin rpy="0 0 0" xyz="0 0 0"/>
             <geometry>
-                <cylinder radius="0.5" length="0.4"/>
+                <cylinder radius="0.5" length="0.5"/>
             </geometry>
         </visual>
@@ -69,5 +69,5 @@
     name="joint_1"
     type="revolute">
-    <origin xyz="0 0 0" rpy="0 0 0" />
+    <origin xyz="0 0 0.25" rpy="0 0 0" />
     <limit effort="1000.0" lower="-3.14" upper="3.14" velocity="0.5" />
     <parent link="base_rotation" />
@@ -142,5 +142,5 @@
     </link>
     <joint name="end" type="fixed">
-        <origin rpy="0 0 0" xyz="0 0 2.5"/>
+        <origin rpy="0 0 0" xyz="0 0 2.4"/>
         <parent link="second_link"/>
         <child link="third_link"/>
